File: SMARTBIKE2_Kicad/SmartBike2/SmartBike2.kicad_pcb (KiCad board)
At the start: 2 copper layers, 106.2 x 115 mm, 91 parts, among them IC1 ESP32-WROVER-B__8MB_, J1 Conn_01x02, J2 RJ45, J3 Conn_01x05, J4 Conn_01x06, J5 Conn_01x08, J6 Conn_01x04, J7 Conn_01x04, Q1 SI2302, Q2 FDN340P, Q3 SI2302, Q4 SI2302, Q5 SI2302, Q6 SI2302, Q7 FDN340P, Q8 SI2302, SW1 SW_Boot, SW2 SW_Reset, U1 MIC5219-3.3YM5, U2 MIC29302WU, U3 NA555D, U4 LM358, U5 NA555D, U6 MIC5219-3.3YM5

Commit message: Arreglo
Parts:
- moved R8 4.21 mm to (196.5, 68.0)
- moved R7 3.58 mm to (191.6, 67.1)
- moved Q3 3.37 mm to (202.8, 57.3)
- moved R12 3.06 mm to (210.0, 73.3)
- moved R35 2.93 mm to (159.4, 117.6)
- moved R29 2.89 mm to (159.5, 121.1)
- moved D4 2.87 mm to (164.5, 121.2)
- moved Q4 2.74 mm to (202.8, 62.8)
- moved J4 2.61 mm to (177.3, 129.0)
- moved R11 2.20 mm to (214.7, 73.2)
- moved R34 2.19 mm to (159.4, 114.1)
- moved R16 2.17 mm to (222.1, 63.3)
- moved Q5 2.05 mm to (202.8, 68.5)
- moved R33 1.22 mm to (159.3, 110.7)
- moved C11 1.16 mm to (210.0, 68.9)
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Other:
- outline, holes or cut-outs redrawn
