File: SMARTBIKE2_Kicad/SmartBike2/SB2_FEED_ALARM/SB2_FEED_ALARM.kicad_sch (KiCad schematic)
At the start: 5 parts, among them J1 Conn_01x08

Commit message: Fase 2 de 3 panel full
+ PCB Acondicionamiento y Módulos

~ Esquemático Luces
~ PCB 3 de 3, Luces
~ Panelización
Other:
- note added: "Conexión a placa con ESP32 y módulos."
Changed lines of the file:
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@@
     (stroke (width 0) (type default))
+  )
+  (text "Conexión a placa con ESP32 y módulos." (at 135.89 109.22 0)
+    (effects (font (size 1.27 1.27)) (justify left bottom))
   )
   (global_label "4.1V" (shape output) (at 168.91 39.37 0) (fields_autoplaced)
@@
     )
   )
-  (global_label "+3.3_2" (shape input) (at 158.75 26.67 90) (fields_autoplaced)
+  (global_label "+3.3_2" (shape output) (at 158.75 26.67 90) (fields_autoplaced)
     (effects (font (size 1.27 1.27)) (justify left))
     (property "Intersheetrefs" "${INTERSHEET_REFS}" (at 158.75 16.9115 90)
