File: SMARTBIKE2_Kicad/SmartBike2/SB2_FEED_ALARM/feeding.kicad_sch (KiCad schematic)
At the start: 18 parts

Commit message: Fase 2 de 3 panel full
+ PCB Acondicionamiento y Módulos

~ Esquemático Luces
~ PCB 3 de 3, Luces
~ Panelización
Changed lines of the file:
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@@
     )
   )
-  (global_label "+3.3_2" (shape input) (at 163.83 76.2 90) (fields_autoplaced)
+  (global_label "+3.3_2" (shape output) (at 163.83 76.2 90) (fields_autoplaced)
     (effects (font (size 1.27 1.27)) (justify left))
     (property "Intersheetrefs" "${INTERSHEET_REFS}" (at 163.83 66.4415 90)
