File: SMARTBIKE2_Kicad/SmartBike2/SB2_LIGTHS/SB2_LIGTHS.kicad_sch (KiCad schematic)
At the start: 7 parts, among them J1 RJ45, Q1 SI2302, Q2 FDN340P

Commit message: PCB 3 de 3
+PCB 3 de 3, Luces

~Panelización
Parts:
- added H1, H2, H3, H4: MountingHole, MountingHole:MountingHole_2.2mm_M2, symbol Mechanical:MountingHole
- added J1: Conn_01x02, Connector_JST:JST_XH_B2B-XH-A_1x02_P2.50mm_Vertical, symbol Connector_Generic:Conn_01x02
- JP1: footprint (none) -> Connector_JST:JST_XH_B2B-XH-A_1x02_P2.50mm_Vertical
- renumbered J1 to J2
Connections:
- net CtrLuces: now also J1.1 (Pin_1)
- net GND: now also J1.2 (Pin_2)
